File: DAQ Case/DAQ Case/DAQ Case.kicad_sch (KiCad schematic)
At the start: 2 parts, among them U1 Teensy4.1

Commit message: add c1 and c0
Connections:
- net pyro_1_cont_out is gone; now on net CP1: U1.11 (9_OUT1C)
- net pyro_2_cont_out is gone; now on net CP2: U1.12 (10_CS_MQSR)
- net CP1: now also A1.1 (D1/TX)
- net CP2: now also A1.2 (D0/RX)
- net RFM95_CS: now also A1.12 (D9)
- net RFM95_INT: now also A1.5 (D2)
- net RFM95_RST: now also A1.13 (D10)
- net buzzerPin: now also A1.6 (D3)
Changed lines of the file:
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@@
+	(wire
+		(pts
+			(xy 231.14 148.59) (xy 256.54 148.59)
+		)
+		(stroke
+			(width 0)
+			(type default)
+		)
+	)
 	(wire
 		(pts
@@
 	(wire
 		(pts
+			(xy 213.36 123.19) (xy 256.54 123.19)
+		)
+		(stroke
+			(width 0)
+			(type default)
+		)
+	)
+	(wire
+		(pts
 			(xy 153.67 140.97) (xy 180.34 140.97)
 		)
@@
 	(wire
 		(pts
+			(xy 231.14 146.05) (xy 256.54 146.05)
+		)
+		(stroke
+			(width 0)
+			(type default)
+		)
+	)
+	(wire
+		(pts
 			(xy 205.74 135.89) (xy 205.74 151.13)
 		)
@@
 	(wire
 		(pts
+			(xy 62.23 91.44) (xy 210.82 91.44)
+		)
+		(stroke
+			(width 0)
+			(type default)
+		)
+	)
+	(wire
+		(pts
 			(xy 256.54 135.89) (xy 205.74 135.89)
 		)
@@
 	(wire
 		(pts
+			(xy 59.69 88.9) (xy 59.69 135.89)
+		)
+		(stroke
+			(width 0)
+			(type default)
+		)
+	)
+	(wire
+		(pts
 			(xy 97.79 185.42) (xy 97.79 187.96)
 		)
@@
 	(wire
 		(pts
+			(xy 213.36 123.19) (xy 213.36 88.9)
+		)
+		(stroke
+			(width 0)
+			(type default)
+		)
+	)
+	(wire
+		(pts
 			(xy 281.94 153.67) (xy 304.8 153.67)
 		)
@@
 	(wire
 		(pts
+			(xy 62.23 133.35) (xy 97.79 133.35)
+		)
+		(stroke
+			(width 0)
+			(type default)
+		)
+	)
+	(wire
+		(pts
 			(xy 153.67 130.81) (xy 180.34 130.81)
 		)
@@
 	(wire
 		(pts
+			(xy 210.82 91.44) (xy 210.82 125.73)
+		)
+		(stroke
+			(width 0)
+			(type default)
+		)
+	)
+	(wire
+		(pts
 			(xy 153.67 153.67) (xy 208.28 153.67)
 		)
@@
 	(wire
 		(pts
+			(xy 59.69 135.89) (xy 97.79 135.89)
+		)
+		(stroke
+			(width 0)
+			(type default)
+		)
+	)
+	(wire
+		(pts
+			(xy 231.14 130.81) (xy 256.54 130.81)
+		)
+		(stroke
+			(width 0)
+			(type default)
+		)
+	)
+	(wire
+		(pts
 			(xy 213.36 143.51) (xy 213.36 158.75)
 		)
@@
 	(wire
 		(pts
+			(xy 213.36 88.9) (xy 59.69 88.9)
+		)
+		(stroke
+			(width 0)
+			(type default)
+		)
+	)
+	(wire
+		(pts
+			(xy 231.14 128.27) (xy 256.54 128.27)
+		)
+		(stroke
+			(width 0)
+			(type default)
+		)
+	)
+	(wire
+		(pts
 			(xy 153.67 135.89) (xy 180.34 135.89)
 		)
@@
 	(wire
 		(pts
+			(xy 62.23 133.35) (xy 62.23 91.44)
+		)
+		(stroke
+			(width 0)
+			(type default)
+		)
+	)
+	(wire
+		(pts
 			(xy 55.88 140.97) (xy 97.79 140.97)
 		)
@@
 	(wire
 		(pts
-			(xy 67.31 133.35) (xy 97.79 133.35)
-		)
-		(stroke
-			(width 0)
-			(type default)
-		)
-	)
-	(wire
-		(pts
 			(xy 200.66 96.52) (xy 200.66 146.05)
 		)
@@
 	(wire
 		(pts
-			(xy 67.31 135.89) (xy 97.79 135.89)
+			(xy 210.82 125.73) (xy 256.54 125.73)
 		)
 		(stroke
@@
 		)
 	)
-	(label "pyro_2_fire_cmd"
-		(at 231.14 151.13 0)
-		(effects
-			(font
-				(size 1.27 1.27)
-			)
-			(justify left bottom)
-		)
-	)
 	(label "RFM95_RST"
 		(at 231.14 148.59 0)
@@
 		)
 	)
-	(label "pyro_2_fire_cmd"
-		(at 231.14 153.67 0)
-		(effects
-			(font
-				(size 1.27 1.27)
-			)
-			(justify left bottom)
-		)
-	)
 	(label "PT_TANK"
 		(at 304.8 153.67 180)
@@
 		)
 	)
-	(label "pyro_2_cont_out"
-		(at 67.31 135.89 0)
-		(effects
-			(font
-				(size 1.27 1.27)
-			)
-			(justify left bottom)
-		)
-	)
 	(label "SERVO3"
 		(at 90.17 120.65 0)
@@
 		)
 	)
+	(label "CP2"
+		(at 67.31 135.89 0)
+		(effects
+			(font
+				(size 1.27 1.27)
+			)
+			(justify left bottom)
+		)
+	)
 	(label "fill_cmd"
 		(at 231.14 133.35 0)
@@
 		)
 	)
+	(label "CP1"
+		(at 67.31 133.35 0)
+		(effects
+			(font
+				(size 1.27 1.27)
+			)
+			(justify left bottom)
+		)
+	)
 	(label "RFM95_CS"
 		(at 231.14 146.05 0)
@@
 		)
 	)
-	(label "pyro_1_cont_out"
-		(at 67.31 133.35 0)
-		(effects
-			(font
-				(size 1.27 1.27)
-			)
-			(justify left bottom)
-		)
-	)
 	(label "radio_volt_mon"
 		(at 67.31 153.67 0)
@@
 		(effects
 			(font
-				(size 1.27 1.27)
-			)
-			(justify left bottom)
-		)
-	)
-	(label "pyro_2_fire_cmd"
-		(at 231.14 156.21 0)
-		(effects
-			(font

Commit message: working live data with everything from the teensy
Connections:
- net SERVO6: now also U1.11 (9_OUT1C); no longer U1.9 (7_RX2_OUT1A)
- net spare_1: now also U1.12 (10_CS_MQSR); no longer U1.10 (8_TX2_IN1)
- net CP1 renamed TSY_RX
- net TSY_RX: now also U1.9 (7_RX2_OUT1A); no longer U1.11 (9_OUT1C)
- net CP2 renamed TSY_TX
- net TSY_TX: now also U1.10 (8_TX2_IN1); no longer U1.12 (10_CS_MQSR)
Changed lines of the file:
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@@
-	(wire
-		(pts
-			(xy 59.69 88.9) (xy 59.69 135.89)
-		)
-		(stroke
-			(width 0)
-			(type default)
-		)
-	)
 	(wire
 		(pts
@@
 	(wire
 		(pts
-			(xy 90.17 128.27) (xy 97.79 128.27)
-		)
-		(stroke
-			(width 0)
-			(type default)
-		)
-	)
-	(wire
-		(pts
 			(xy 153.67 138.43) (xy 180.34 138.43)
 		)
@@
 	(wire
 		(pts
+			(xy 90.17 133.35) (xy 97.79 133.35)
+		)
+		(stroke
+			(width 0)
+			(type default)
+		)
+	)
+	(wire
+		(pts
 			(xy 281.94 143.51) (xy 304.8 143.51)
 		)
@@
 	(wire
 		(pts
+			(xy 62.23 128.27) (xy 97.79 128.27)
+		)
+		(stroke
+			(width 0)
+			(type default)
+		)
+	)
+	(wire
+		(pts
 			(xy 213.36 123.19) (xy 213.36 88.9)
 		)
@@
 	(wire
 		(pts
-			(xy 62.23 133.35) (xy 97.79 133.35)
-		)
-		(stroke
-			(width 0)
-			(type default)
-		)
-	)
-	(wire
-		(pts
 			(xy 153.67 130.81) (xy 180.34 130.81)
 		)
@@
 	(wire
 		(pts
+			(xy 78.74 135.89) (xy 97.79 135.89)
+		)
+		(stroke
+			(width 0)
+			(type default)
+		)
+	)
+	(wire
+		(pts
 			(xy 210.82 140.97) (xy 256.54 140.97)
 		)
@@
 	(wire
 		(pts
-			(xy 59.69 135.89) (xy 97.79 135.89)
-		)
-		(stroke
-			(width 0)
-			(type default)
-		)
-	)
-	(wire
-		(pts
 			(xy 231.14 130.81) (xy 256.54 130.81)
 		)
@@
 	(wire
 		(pts
+			(xy 62.23 91.44) (xy 62.23 128.27)
+		)
+		(stroke
+			(width 0)
+			(type default)
+		)
+	)
+	(wire
+		(pts
 			(xy 153.67 148.59) (xy 203.2 148.59)
 		)
@@
 	(wire
 		(pts
-			(xy 67.31 130.81) (xy 97.79 130.81)
-		)
-		(stroke
-			(width 0)
-			(type default)
-		)
-	)
-	(wire
-		(pts
-			(xy 62.23 133.35) (xy 62.23 91.44)
+			(xy 59.69 88.9) (xy 59.69 130.81)
 		)
 		(stroke
@@
 		(pts
 			(xy 210.82 125.73) (xy 256.54 125.73)
+		)
+		(stroke
+			(width 0)
+			(type default)
+		)
+	)
+	(wire
+		(pts
+			(xy 59.69 130.81) (xy 97.79 130.81)
 		)
 		(stroke
@@
 		)
 	)
-	(label "SERVO6"
-		(at 90.17 128.27 0)
-		(effects
-			(font
-				(size 1.27 1.27)
-			)
-			(justify left bottom)
-		)
-	)
 	(label "0_TSY"
 		(at 90.17 110.49 0)
@@
 		)
 	)
-	(label "CP2"
-		(at 231.14 123.19 0)
-		(effects
-			(font
-				(size 1.27 1.27)
-			)
-			(justify left bottom)
-		)
-	)
 	(label "PT_TANK"
 		(at 304.8 153.67 180)
@@
 		)
 	)
-	(label "CP2"
-		(at 67.31 135.89 0)
-		(effects
-			(font
-				(size 1.27 1.27)
+	(label "TSY_TX"
+		(at 90.17 130.81 0)
+		(effects
+			(font
+				(size 1.27 1.27)
+				(color 0 0 255 1)
 			)
 			(justify left bottom)
@@
 		)
 	)
-	(label "CP1"
-		(at 67.31 133.35 0)
-		(effects
-			(font
-				(size 1.27 1.27)
+	(label "TSY_RX"
+		(at 90.17 128.27 0)
+		(effects
+			(font
+				(size 1.27 1.27)
+				(color 0 0 255 1)
 			)
 			(justify left bottom)
@@
 		)
 	)
+	(label "TSY_RX"
+		(at 231.14 125.73 0)
+		(effects
+			(font
+				(size 1.27 1.27)
+				(color 0 0 255 1)
+			)
+			(justify left bottom)
+		)
+	)
 	(label "RADIO_LED"
 		(at 304.8 143.51 180)
@@
 		)
 	)
+	(label "spare_1"
+		(at 78.74 135.89 0)
+		(effects
+			(font
+				(size 1.27 1.27)
+				(color 0 0 255 1)
+			)
+			(justify left bottom)
+		)
+	)
 	(label "pyro_2_fire"
 		(at 180.34 166.37 180)
@@
 		)
 	)
+	(label "TSY_TX"
+		(at 231.14 123.19 0)
+		(effects
+			(font
+				(size 1.27 1.27)
+				(color 0 0 255 1)
+			)
+			(justify left bottom)
+		)
+	)
 	(label "pt_5"
 		(at 180.34 123.19 180)
@@
 		)
 	)
-	(label "CP1"
-		(at 231.14 125.73 0)
-		(effects
-			(font
-				(size 1.27 1.27)
-			)
-			(justify left bottom)
-		)
-	)
 	(label "lc_high"
 		(at 304.8 148.59 180)
@@
 		)
 	)
+	(label "SERVO6"
+		(at 90.17 133.35 0)
+		(effects
+			(font
+				(size 1.27 1.27)
+				(color 0 0 255 1)
+			)
+			(justify left bottom)
+		)
+	)
 	(label "mov_cmd"
 		(at 231.14 138.43 0)
@@
 		(effects
 			(font
-				(size 1.27 1.27)
-			)
-			(justify left bottom)
-		)
-	)
-	(label "spare_1"
-		(at 67.31 130.81 0)
-		(effects
-			(font
